Commit message: first stanfing motion

File: urdf/bipedal_plateform/urdf/robot.urdf (robot description, URDF)
Before this commit: robot urdf, 17 links, 16 joints
Links:
- added link torso_assembly, mass 1e-09; collision mesh filename=package://assets/bearing_holder_upperbody.stl; collision mesh filename=package://assets/bearing_holder_upperbody.stl
Joints:
- added joint upper_body: type fixed, parent torso_subassembly, child torso_assembly, origin xyz=-0.0205415 4.03795e-07 0.036034 rpy=-3.14159 -7.46619e-17 1.59378e-17, axis 0 0 1, limit effort=10 velocity=10
- joint anklex_left: origin xyz=7.77156e-15 -0.01594 0.02 rpy=1.5708 -1.27182 7.14944e-14 -> xyz=7.99361e-15 -0.01594 0.02 rpy=-1.5708 -1.51155 -3.14159
- joint anklex_right: origin xyz=-5.21805e-15 -0.01594 0.02 rpy=1.5708 1.37363 -1.82916e-13 -> xyz=-5.55112e-15 -0.01594 0.02 rpy=1.5708 1.56918 -2.91336e-11
- joint ankley_left: origin xyz=6.66134e-16 -0.26 -0.02 rpy=-8.03076e-15 -4.82577e-15 -1.10322 -> xyz=-3.88578e-16 -0.26 -0.02 rpy=-1.75167e-15 -2.14857e-15 -1.50866
- joint ankley_right: origin xyz=-0.158187 -0.206341 0.02 rpy=3.14159 -8.93239e-15 0.907084 -> xyz=-0.218697 -0.140611 0.02 rpy=3.14159 -6.83356e-15 1.16506
- joint hipx_left: origin xyz=-0.01897 0.0289 -0.09689 rpy=0.313623 0.0639766 -2.75553 -> xyz=-0.01897 0.0289 -0.09689 rpy=-0.00578336 0.31982 2.1331
- joint hipx_right: origin xyz=-0.01897 -0.0289 -0.09689 rpy=-0.237662 0.216147 -2.99762 -> xyz=-0.01897 -0.0289 -0.09689 rpy=-0.0611181 0.314174 -2.34698
- joint hipy_left: origin xyz=0.012638 0.0276823 -0.112055 rpy=1.7327 -1.14007 2.56649 -> xyz=0.012638 0.0276823 -0.112055 rpy=1.72118 -1.1049 2.57926
- joint hipy_right: origin xyz=0.012638 -0.0276823 -0.112055 rpy=-1.65071 0.567773 -2.75687 -> xyz=0.012638 -0.0276823 -0.112055 rpy=-1.64283 0.361997 -2.73937
- joint hipz_left: origin xyz=-0.00081771 0.13316 0.04164 rpy=-0.104044 0.0956642 0.716096 -> xyz=-0.00081771 0.13316 0.04164 rpy=-0.0308207 0.13784 1.32527
- joint hipz_right: origin xyz=-0.00081771 -0.133159 0.04164 rpy=0.120992 0.073012 -0.51559 -> xyz=-0.00081771 -0.133159 0.04164 rpy=0.0465927 0.133363 -1.20873
- joint knee_left: origin xyz=-0.17 -0.294449 -0.0305 rpy=-1.56672e-14 1.36641e-14 -1.71007 -> xyz=-0.17 -0.294449 -0.0305 rpy=1.04567e-14 2.64358e-14 -1.47151
- joint knee_right: origin xyz=0.17 0.294449 -0.0305 rpy=3.14159 -1.42168e-13 -0.93033 -> xyz=0.17 0.294449 -0.0305 rpy=-3.14159 -1.47653e-14 -0.46045

File: urdf/humanoid_v0/urdf/robot.urdf (robot description, URDF)
Before this commit: robot onshape, 33 links, 32 joints
Links:
- link foot: mass 0.10323152601569812736 -> 0.10864739156748566551
- link foot_2: mass 0.10323152601569812736 -> 0.10864739156748566551
- link hipx: mass 0.40837828065714160131 -> 0.4083782806571415458
- link hipx_2: mass 0.40837828065714160131 -> 0.4083782806571415458
- link hipz: mass 0.23297090955878962948 -> 0.23297090955878965723
- link hipz_2: mass 0.23297090955878962948 -> 0.23297090955878965723
- link rmdx43: mass 0.30000000000000004441 -> 0.2999999999999999889
- link rmdx43_2: mass 0.30000000000000004441 -> 0.2999999999999999889
- link rmdx43_3: mass 0.30000000000000004441 -> 0.2999999999999999889
- link rmdx43_4: mass 0.30000000000000004441 -> 0.2999999999999999889
- link torso_base: mass 0.47534767265056637742 -> 0.47534767265056632191
- link ujoint: mass 0.064941739054599462166 -> 0.064941739054599448289
- link ujoint_2: mass 0.064941739054599462166 -> 0.064941739054599448289
Joints:
- joint anklex_left: origin xyz=-0.010036795405957782412 0.017299212062372393284 -2.7755575615628913511e-17 rpy=1.570796326794896558 5.1580029225031729764e-09 -1.0450718614477501056 -> xyz=-0.010036795405957782412 0.017299212062372615328 -2.7755575615628913511e-17 rpy=1.570796326794896558 5.1580029225031738036e-09 -1.0450718614477498836
- joint anklex_right: origin xyz=-0.010036795405958004457 0.017299212062372393284 -1.3877787807814456755e-17 rpy=1.5707963267948981123 6.0492654793778970011e-15 -1.0450718614477441104 -> xyz=-0.010036795405957948946 0.017299212062372615328 -1.3877787807814456755e-17 rpy=1.5707963267948981123 6.0492654793778962122e-15 -1.0450718614477438884
- joint foot_left_frame: origin xyz=-0.023424822443902426627 -2.7755575615628913511e-17 -0.0060508435686524308927 rpy=-1.286607748282698211e-25 1.570796326794896558 0 -> xyz=-0.040000000000000146549 -1.3877787807814456755e-17 -0.0060508435686522782371 rpy=1.2655393534870346686e-24 1.570796326794896558 0
- joint foot_right_frame: origin xyz=-0.023424822443902426627 -2.7755575615628913511e-17 -0.0060508435686524031372 rpy=-8.9378788990096449613e-33 1.570796326794896558 0 -> xyz=-0.040000000000000257572 -1.3877787807814456755e-17 -0.0060508435686522782371 rpy=-2.1672957339748004381e-31 1.570796326794896558 0
